File: sync.kicad_sch (KiCad schematic)
At the start: 29 parts, among them J2 ALTOSC, J3 DE15_VGA, U11 74LS20(ЛА1), U12 74LS02(ЛЕ1), U12 74LS21(ЛИ6), U17 74LS163(ИЕ18), U18 74LS175(ТМ8), U19 74LS93(ИЕ5), U20 TC4426, U21 74LS163(ИЕ18), U22 74LS00(ЛА3), U22 74LS163(ИЕ18), U23 74HCT4040, U24 74LS377(ИР27), U25 74LS377(ИР27), U26 74LS243(ИП7), U27 74LS166(ИР10), U28 74LS166(ИР10), U3 74LS02(ЛЕ1), U5 74LS04(ЛН1), U6 74LS08(ЛИ1), U9 74LS10(ЛА4), X1 25.175 MHz

Commit message: fix VGA output resistor values
Parts:
- R10: value 560 -> 360
- R5, R6: value 910 -> 620
- R7: value 1k3 -> 910
- R8: value 680 -> 470
- R9: value 2k7 -> 1k8
Changed lines of the file:
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@@
       (effects (font (size 1.27 1.27)) (justify right))
     )
-    (property "Value" "2k7" (at 215.9 134.62 90)
+    (property "Value" "1k8" (at 215.9 134.62 90)
       (effects (font (size 1.27 1.27)))
     )
@@
       (effects (font (size 1.27 1.27)) (justify right))
     )
-    (property "Value" "1k3" (at 207.01 137.16 90)
+    (property "Value" "910" (at 207.01 137.16 90)
       (effects (font (size 1.27 1.27)))
     )
@@
       (effects (font (size 1.27 1.27)) (justify right))
     )
-    (property "Value" "680" (at 207.01 144.78 90)
+    (property "Value" "470" (at 207.01 144.78 90)
       (effects (font (size 1.27 1.27)))
     )
@@
       (effects (font (size 1.27 1.27)) (justify right))
     )
-    (property "Value" "560" (at 215.9 142.24 90)
+    (property "Value" "360" (at 215.9 142.24 90)
       (effects (font (size 1.27 1.27)))
     )
@@
       (effects (font (size 1.27 1.27)) (justify right))
     )
-    (property "Value" "910" (at 198.12 147.32 90)
+    (property "Value" "620" (at 198.12 147.32 90)
       (effects (font (size 1.27 1.27)))
     )
@@
       (effects (font (size 1.27 1.27)) (justify right))
     )
-    (property "Value" "910" (at 198.12 139.7 90)
-      (effects (font (size 1.27 1.27)))
-    )
+    (property "Value" "620" (at 198.12 139.7 90)
+      (effects (font (size 1.27 1.27)))
+    )

Commit message: video byte reverse
Connections:
- net VD0: now also U24.3 (D0), U25.3 (D0); no longer U24.18 (D7), U25.18 (D7)
- net VD1: now also U24.4 (D1), U25.4 (D1); no longer U24.17 (D6), U25.17 (D6)
- net VD2: now also U24.7 (D2), U25.7 (D2); no longer U24.14 (D5), U25.14 (D5)
- net VD3: now also U24.8 (D3), U25.8 (D3); no longer U24.13 (D4), U25.13 (D4)
- net VD4: now also U24.13 (D4), U25.13 (D4); no longer U24.8 (D3), U25.8 (D3)
- net VD5: now also U24.14 (D5), U25.14 (D5); no longer U24.7 (D2), U25.7 (D2)
- net VD6: now also U24.17 (D6), U25.17 (D6); no longer U24.4 (D1), U25.4 (D1)
- net VD7: now also U24.18 (D7), U25.18 (D7); no longer U24.3 (D0), U25.3 (D0)

Commit message: fix RAM multiplexers connections
Connections:
- no-connect marks 18 -> 17
Changed lines of the file:
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@@
   (no_connect (at 50.8 119.38))
   (no_connect (at 50.8 121.92))
-  (no_connect (at 55.88 109.22))
   (no_connect (at 261.62 147.32))
   (no_connect (at 50.8 114.3))
@@
     (stroke (width 0) (type default))
   )
-  (wire (pts (xy 50.8 109.22) (xy 55.88 109.22))
-    (stroke (width 0) (type default))
-  )
   (wire (pts (xy 19.05 124.46) (xy 25.4 124.46))
     (stroke (width 0) (type default))
@@
   (label "RED" (at 189.23 134.62 180) (fields_autoplaced)
     (effects (font (size 1.27 1.27)) (justify right bottom))
-  )
-  (label "T3" (at 52.07 109.22 0) (fields_autoplaced)
-    (effects (font (size 1.27 1.27)) (justify left bottom))
   )
   (label "VD7" (at 194.31 44.45 0) (fields_autoplaced)
@@
     )
   )
+  (global_label "T3" (shape output) (at 50.8 109.22 0) (fields_autoplaced)
+    (effects (font (size 1.27 1.27)) (justify left))
+    (property "Intersheetrefs" "${INTERSHEET_REFS}" (at 55.9623 109.22 0)
+      (effects (font (size 1.27 1.27)) (justify left) hide)
+    )
+  )
