File: io.kicad_sch (KiCad schematic)
At the start: 18 parts, among them J10 SEGA, J11 PS/2, J12 UART, U15 74LS14(ТЛ2), U16 74LS74(ТМ2), U3 74LS04(ЛН1), U33 74LS02(ЛЕ1), U45 8255A(КР580ВВ55А), U46 AT90S2313, U47 8251A(КР580ВВ51А), U5 74LS08(ЛИ1), U5 74LS10(ЛА4), U6 74LS08(ЛИ1), U7 74LS74(ТМ2), U8 74LS00(ЛА3), U9 74LS00(ЛА3)

Commit message: fix RAM transceiver connections
Parts:
- removed unit 3 of U8
Connections:
- no-connect marks 16 -> 15
Other:
- moved on the sheet: U8B
Changed lines of the file:
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@@
   (no_connect (at 111.76 182.88))
   (no_connect (at 154.94 68.58))
-  (no_connect (at 157.48 154.94))
   (no_connect (at 154.94 66.04))
   (no_connect (at 124.46 40.64))
@@
     )
   )
-  (symbol (lib_id "74xx:74LS00") (at 149.86 154.94 0) (unit 2)
-    (in_bom yes) (on_board yes) (dnp no) (fields_autoplaced)
-    (property "Reference" "U8" (at 149.8517 146.05 0)
-      (effects (font (size 1.27 1.27)))
-    )
-    (property "Value" "74LS00(ЛА3)" (at 149.8517 148.59 0)
-      (effects (font (size 1.27 1.27)))
-    )
-    (property "Footprint" "Package_DIP:DIP-14_W7.62mm" (at 149.86 154.94 0)
-      (effects (font (size 1.27 1.27)) hide)
-    )
-    (property "Datasheet" "http://www.ti.com/lit/gpn/sn74ls00" (at 149.86 154.94 0)
+  (symbol (lib_id "74xx:74LS00") (at 149.86 170.18 0) (unit 2)
+    (in_bom yes) (on_board yes) (dnp no) (fields_autoplaced)
+    (property "Reference" "U8" (at 149.8517 161.29 0)
+      (effects (font (size 1.27 1.27)))
+    )
+    (property "Value" "74LS00(ЛА3)" (at 149.8517 163.83 0)
+      (effects (font (size 1.27 1.27)))
+    )
+    (property "Footprint" "Package_DIP:DIP-14_W7.62mm" (at 149.86 170.18 0)
+      (effects (font (size 1.27 1.27)) hide)
+    )
+    (property "Datasheet" "http://www.ti.com/lit/gpn/sn74ls00" (at 149.86 170.18 0)
       (effects (font (size 1.27 1.27)) hide)
     )
@@
         (path "/76485272-58b9-4241-940e-8879fa844c96/0567776f-ec27-40d8-a046-f38d0368ad09"
           (reference "U16") (unit 1)
-        )
-      )
-    )
-  )
-  (symbol (lib_id "power:+5V") (at 142.24 157.48 90) (unit 1)
-    (in_bom yes) (on_board yes) (dnp no)
-    (property "Reference" "#PWR02" (at 146.05 157.48 0)
-      (effects (font (size 1.27 1.27)) hide)
-    )
-    (property "Value" "+5V" (at 137.16 157.48 90)
-      (effects (font (size 1.27 1.27)))
-    )
-    (property "Footprint" "" (at 142.24 157.48 0)
-      (effects (font (size 1.27 1.27)) hide)
-    )
-    (property "Datasheet" "" (at 142.24 157.48 0)
-      (effects (font (size 1.27 1.27)) hide)
-    )
-    (pin "1")
-    (instances
-      (project "pac80"
-        (path "/76485272-58b9-4241-940e-8879fa844c96/bd8626b9-ceff-4d5c-a266-06111337714c"
-          (reference "#PWR02") (unit 1)
-        )
-        (path "/76485272-58b9-4241-940e-8879fa844c96/e05dffe5-a8ce-4bdd-b0f4-f983b256ebc2"
-          (reference "#PWR055") (unit 1)
-        )
-        (path "/76485272-58b9-4241-940e-8879fa844c96/e5b989ce-1e05-4470-9bcf-aea14f9cddaf"
-          (reference "#PWR074") (unit 1)
-        )
-        (path "/76485272-58b9-4241-940e-8879fa844c96/3455005e-76fb-4d3b-af2a-bae2cb5cdaf9"
-          (reference "#PWR0142") (unit 1)
-        )
-        (path "/76485272-58b9-4241-940e-8879fa844c96/0567776f-ec27-40d8-a046-f38d0368ad09"
-          (reference "#PWR0284") (unit 1)
         )
       )
@@
     )
   )
-  (symbol (lib_id "74xx:74LS00") (at 149.86 170.18 0) (unit 3)
-    (in_bom yes) (on_board yes) (dnp no)
-    (property "Reference" "U8" (at 149.8517 161.29 0)
-      (effects (font (size 1.27 1.27)))
-    )
-    (property "Value" "74LS00(ЛА3)" (at 149.8517 163.83 0)
-      (effects (font (size 1.27 1.27)))
-    )
-    (property "Footprint" "Package_DIP:DIP-14_W7.62mm" (at 149.86 170.18 0)
-      (effects (font (size 1.27 1.27)) hide)
-    )
-    (property "Datasheet" "http://www.ti.com/lit/gpn/sn74ls00" (at 149.86 170.18 0)
-      (effects (font (size 1.27 1.27)) hide)
-    )
-    (pin "1")
-    (pin "2")
-    (pin "3")
-    (pin "4")
-    (pin "5")
-    (pin "6")
-    (pin "10")
-    (pin "8")
-    (pin "9")
-    (pin "11")
-    (pin "12")
-    (pin "13")
-    (pin "14")
-    (pin "7")
-    (instances
-      (project "pac80"
-        (path "/76485272-58b9-4241-940e-8879fa844c96/e5b989ce-1e05-4470-9bcf-aea14f9cddaf"
-          (reference "U8") (unit 3)
-        )
-        (path "/76485272-58b9-4241-940e-8879fa844c96/3455005e-76fb-4d3b-af2a-bae2cb5cdaf9"
-          (reference "U2") (unit 3)
-        )
-        (path "/76485272-58b9-4241-940e-8879fa844c96/34cd57db-2a21-4ed7-a0b6-b6a247ac7439"
-          (reference "U2") (unit 3)
-        )
-        (path "/76485272-58b9-4241-940e-8879fa844c96/0567776f-ec27-40d8-a046-f38d0368ad09"
-          (reference "U2") (unit 3)
-        )
-      )
-    )
-  )
   (symbol (lib_id "power:+5V") (at 238.76 91.44 270) (unit 1)
     (in_bom yes) (on_board yes) (dnp no)
@@
         )
       )
-    )
-  )
-  (symbol (lib_id "power:+5V") (at 142.24 152.4 90) (unit 1)
-    (in_bom yes) (on_board yes) (dnp no)
-    (property "Reference" "#PWR02" (at 146.05 152.4 0)
-      (effects (font (size 1.27 1.27)) hide)
-    )
-    (property "Value" "+5V" (at 137.16 152.4 90)
-      (effects (font (size 1.27 1.27)))
-    )
-    (property "Footprint" "" (at 142.24 152.4 0)
-      (effects (font (size 1.27 1.27)) hide)
-    )
-    (property "Datasheet" "" (at 142.24 152.4 0)
-      (effects (font (size 1.27 1.27)) hide)
-    )
-    (pin "1")
-    (instances
-      (project "pac80"
-        (path "/76485272-58b9-4241-940e-8879fa844c96/bd8626b9-ceff-4d5c-a266-06111337714c"
-          (reference "#PWR02") (unit 1)
-        )
-        (path "/76485272-58b9-4241-940e-8879fa844c96/e05dffe5-a8ce-4bdd-b0f4-f983b256ebc2"
-          (reference "#PWR055") (unit 1)
-        )
-        (path "/76485272-58b9-4241-940e-8879fa844c96/e5b989ce-1e05-4470-9bcf-aea14f9cddaf"
-          (reference "#PWR074") (unit 1)
-        )
-        (path "/76485272-58b9-4241-940e-8879fa844c96/3455005e-76fb-4d3b-af2a-bae2cb5cdaf9"
-          (reference "#PWR0141") (unit 1)
-        )
-        (path "/76485272-58b9-4241-940e-8879fa844c96/0567776f-ec27-40d8-a046-f38d0368ad09"
-          (reference "#PWR0283") (unit 1)
-        )
-      )
