File: cpu.kicad_sch (KiCad schematic)
At the start: 21 parts, among them J5 CF, J6 CFPWR, J7 EXT0, J8 EXT1, J9 EXT2, SW1 RESET, U10 74LS14(ТЛ2), U13 74LS32(ЛЛ1), U25 74LS245(АП6), U3 74LS04(ЛН1), U39 8080A(КР580ВМ80А), U4 74LS08(ЛИ1), U42 74LS241(АП4), U43 74LS241(АП4), U44 74LS155(ИД4), U8 74LS175(ТМ8)

Commit message: fix VGA output resistor values
Changed lines of the file:
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@@
-    (stroke (width 0) (type default))
-  )
-  (wire (pts (xy 88.9 173.99) (xy 93.98 173.99))
     (stroke (width 0) (type default))
   )
@@
     (effects (font (size 1.27 1.27)) (justify left bottom))
   )
-  (label "~{OUT}" (at 127 86.36 0) (fields_autoplaced)
-    (effects (font (size 1.27 1.27)) (justify left bottom))
-  )
   (label "D4" (at 223.52 80.01 0) (fields_autoplaced)
     (effects (font (size 1.27 1.27)) (justify left bottom))
@@
   )
   (label "~{MEMR}" (at 88.9 128.27 0) (fields_autoplaced)
-    (effects (font (size 1.27 1.27)) (justify left bottom))
-  )
-  (label "~{OUT}" (at 88.9 173.99 0) (fields_autoplaced)
     (effects (font (size 1.27 1.27)) (justify left bottom))
   )
@@
     )
   )
+  (global_label "~{OUT}" (shape input) (at 93.98 173.99 180) (fields_autoplaced)
+    (effects (font (size 1.27 1.27)) (justify right))
+    (property "Intersheetrefs" "${INTERSHEET_REFS}" (at 87.3662 173.99 0)
+      (effects (font (size 1.27 1.27)) (justify right) hide)
+    )
+  )

Commit message: fix power-on-reset circuit
Parts:
- C4: value 0.1u -> 1u
- R3: value 100k -> 1M
Changed lines of the file:
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@@
       (effects (font (size 1.27 1.27)) (justify right))
     )
-    (property "Value" "0.1u" (at 33.02 162.5536 0)
+    (property "Value" "1u" (at 33.02 162.5536 0)
       (effects (font (size 1.27 1.27)) (justify right))
     )
@@
       (effects (font (size 1.27 1.27)))
     )
-    (property "Value" "100k" (at 24.257 152.4 90)
-      (effects (font (size 1.27 1.27)))
-    )
+    (property "Value" "1M" (at 24.257 152.4 90)
+      (effects (font (size 1.27 1.27)))
+    )
