File: power.kicad_sch (KiCad schematic)
At the start: 79 parts, among them J1 USB_B, U1 74LS00(ЛА3), U12 74LS20(ЛА1), U20 74LS02(ЛЕ1), U22 74LS10(ЛА4), U24 74LS32(ЛЛ1), U31 74LS74(ТМ2), U33 74LS02(ЛЕ1), U38 74LS32(ЛЛ1), U40 74LS14(ТЛ2), U41 74LS00(ЛА3), U42 74LS08(ЛИ1), U43 74LS21(ЛИ6), U46 74LS74(ТМ2), U5 74LS04(ЛН1), U6 74LS08(ЛИ1), U8 MC34063AP

Commit message: update Zener diode
Parts:
- D3: value BZX55C11 -> BZX55C10
Changed lines of the file:
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@@
   (symbol (lib_id "Diode:BZV55C11") (at 125.73 46.99 180) (unit 1)
     (in_bom yes) (on_board yes) (dnp no) (fields_autoplaced)
-    (property "Reference" "D3" (at 125.73 41.91 0)
+    (property "Reference" "D3" (at 125.73 40.64 0)
       (effects (font (size 1.27 1.27)))
     )
-    (property "Value" "BZX55C11" (at 125.73 44.45 0)
+    (property "Value" "BZX55C10" (at 125.73 43.18 0)
       (effects (font (size 1.27 1.27)))
     )
